File: STM32H733.kicad_sch (KiCad schematic)
At the start: 85 parts, among them IC1 AT7456E, J1 USB, J2 DJI, J3 SWD, J4 CAM, J6 VTX, J7 GPS, J8 ESC, J9 ELRS, U1 STM32H733VGTx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

Commit message: New Layout designed
Signed-off-by: Asraful Islam Taj <asraful.islam.taj@gmail.com>
Parts:
- removed D1: BAT54C, Package_TO_SOT_SMD:SOT-23, symbol Diode:BAT54C
- added D1, D2: 1N5819WS, Diode_SMD:D_SOD-323, symbol Diode:1N5819WS
- C46: footprint Capacitor_SMD:C_0603_1608Metric -> Capacitor_SMD:C_0402_1005Metric
Connections:
- net +5VUSB: now also D2.2 (A)
- net +B5V: now also D1.2 (A)
- net GPS_USART1_RX: now also U1.55 (PD8); no longer U1.56 (PD9)
- net GPS_USART1_TX: now also U1.56 (PD9); no longer U1.55 (PD8)
- net RC_USART2_RX: now also J9.2 (Pin_2); no longer J9.1 (Pin_1)
- net RC_USART2_TX: now also J9.1 (Pin_1); no longer J9.2 (Pin_2)
- net at C3.1, U3.1 (IN), U3.3 (EN): now also D1.1 (K), D2.1 (K)
